Commit message: Refactor robot odometry and Arduino bridge nodes for improved functionality and safety
- Updated `odom_node.py` to implement encoder-based odometry calculations, enhancing accuracy in robot positioning.
- Introduced new parameters for wheel diameter, separation, and ticks per revolution in `EncoderOdomNode`.
- Modified the odometry publishing mechanism to include covariance for better state estimation.
- Enhanced `arduino_bridge.py` to support encoder data publishing and improved serial connection handling.
- Implemented USB reset functionality for Arduino to ensure reliable communication.
- Added safety features in `safety_node.py` to monitor obstacles using LIDAR data and prevent collisions.
- Refactored command publishing to ensure safe commands are sent to the robot based on obstacle detection.
- Introduced a watchdog mechanism to monitor the health of the IMU and encoder data streams.
- Created a new `teleop_key` package for keyboard teleoperation, including necessary initialization files.

File: robot_ws/src/robot_description/urdf/robot.urdf.xacro (robot description, xacro)
@@ -1,27 +1,8 @@
 <?xml version="1.0"?>
-<robot name="delivery_robot" xmlns:xacro="http://www.ros.org/wiki/xacro">
-  <!--
-    robot_urdf.xacro — Elegoo Smart Car base
-    Frames:
-      base_footprint  (ground projection, odom → here via EKF)
-      base_link       (robot body centre)
-      laser           (RPLidar A1)
-      imu_link        (MPU6050 on Arduino Uno)
-      camera_link     (Pi Camera — add later for QR/ArUco)
-  -->
-  <!-- ============================================================ -->
-  <!-- BASE FOOTPRINT — ground plane projection                      -->
-  <!-- ============================================================ -->
-  <link name="base_footprint"/>
-  <joint name="base_footprint_to_base_link" type="fixed">
-    <parent link="base_footprint"/>
-    <child link="base_link"/>
-    <origin xyz="0 0 0.04" rpy="0 0 0"/>
-    <!-- 0.04m = approx height of Elegoo chassis off ground -->
-  </joint>
-  <!-- ============================================================ -->
-  <!-- BASE LINK — robot body                                        -->
-  <!-- Elegoo Smart Car chassis: ~20cm x 14cm                       -->
-  <!-- ============================================================ -->
+<robot name="delivery_robot"
+       xmlns:xacro="http://www.ros.org/wiki/xacro">
+  <!-- ========================================================== -->
+  <!-- BASE LINK                                                   -->
+  <!-- ========================================================== -->
   <link name="base_link">
     <visual>
@@ -40,18 +21,21 @@
     <inertial>
       <mass value="0.8"/>
-      <!-- Simple box inertia for ~0.8kg robot -->
-      <inertia ixx="0.001" ixy="0" ixz="0"
-               iyy="0.001" iyz="0"
-               izz="0.002"/>
+      <inertia
+        ixx="0.001"
+        ixy="0"
+        ixz="0"
+        iyy="0.001"
+        iyz="0"
+        izz="0.002"/>
     </inertial>
   </link>
-  <!-- ============================================================ -->
-  <!-- LIDAR — RPLidar A1                                           -->
-  <!-- Mounted on top centre of chassis                             -->
-  <!-- ============================================================ -->
+  <!-- ========================================================== -->
+  <!-- RPLIDAR A1                                                  -->
+  <!-- ========================================================== -->
   <link name="laser">
     <visual>
       <geometry>
-        <cylinder radius="0.035" length="0.04"/>
+        <cylinder radius="0.035"
+                  length="0.04"/>
       </geometry>
       <material name="black">
@@ -60,14 +44,15 @@
     </visual>
   </link>
-  <joint name="base_link_to_laser" type="fixed">
+  <joint name="base_link_to_laser"
+         type="fixed">
     <parent link="base_link"/>
     <child link="laser"/>
-    <!-- Centred on top of chassis, adjust x/y if your LiDAR is offset -->
-    <origin xyz="0.0 0.0 0.065" rpy="0 0 0"/>
+    <origin
+      xyz="0.0 0.0 0.065"
+      rpy="0 0 0"/>
   </joint>
-  <!-- ============================================================ -->
-  <!-- IMU LINK — MPU6050 on Arduino Uno                            -->
-  <!-- Arduino sits on chassis, MPU6050 roughly at centre           -->
-  <!-- ============================================================ -->
+  <!-- ========================================================== -->
+  <!-- MPU6050                                                     -->
+  <!-- ========================================================== -->
   <link name="imu_link">
     <visual>
@@ -80,15 +65,15 @@
     </visual>
   </link>
-  <joint name="base_link_to_imu" type="fixed">
+  <joint name="base_link_to_imu"
+         type="fixed">
     <parent link="base_link"/>
     <child link="imu_link"/>
-    <!-- MPU6050 is roughly at the centre of the Arduino board -->
-    <!-- Adjust if your Arduino is offset from chassis centre   -->
-    <origin xyz="0.0 0.0 0.03" rpy="0 0 0"/>
+    <origin
+      xyz="0.0 0.0 0.03"
+      rpy="0 0 0"/>
   </joint>
-  <!-- ============================================================ -->
-  <!-- CAMERA LINK — Pi Camera (placeholder for Phase 4)           -->
-  <!-- Will be used for QR code recipient verification             -->
-  <!-- ============================================================ -->
+  <!-- ========================================================== -->
+  <!-- CAMERA                                                      -->
+  <!-- ========================================================== -->
   <link name="camera_link">
     <visual>
@@ -101,35 +86,11 @@
     </visual>
   </link>
-  <joint name="base_link_to_camera" type="fixed">
+  <joint name="base_link_to_camera"
+         type="fixed">
     <parent link="base_link"/>
     <child link="camera_link"/>
-    <!-- Front of robot, facing forward, at top -->
-    <origin xyz="0.10 0.0 0.06" rpy="0 0 0"/>
+    <origin
+      xyz="0.10 0.0 0.06"
+      rpy="0 0 0"/>
   </joint>
 </robot>
-<!-- <?xml version="1.0"?>
-<robot name="my_robot" xmlns:xacro="http://www.ros.org/wiki/xacro">
-  <!-- BASE FOOTPRINT -->
-  <link name="base_footprint"/>
-  <!-- BASE LINK -->
-  <link name="base_link"/>
-  <joint name="base_footprint_to_base_link" type="fixed">
-    <parent link="base_footprint"/>
-    <child link="base_link"/>
-    <origin xyz="0 0 0" rpy="0 0 0"/>
-  </joint>
-  <!-- LIDAR -->
-  <link name="laser"/>
-  <joint name="base_link_to_laser" type="fixed">
-    <parent link="base_link"/>
-    <child link="laser"/>
-    <origin xyz="0 0 0.15" rpy="0 0 0"/>
-  </joint>
-  <!-- IMU LINK -->
-  <link name="imu_link"/>
-  <joint name="base_link_to_imu" type="fixed">
-    <parent link="base_link"/>
-    <child link="imu_link"/>
-    <origin xyz="0 0 0.05" rpy="0 0 0"/>
-  </joint>
-</robot> -->

Commit message: added autonomous robot movement with obstacles avoidance - added ultrasonic sensor for lower obstacles avoidance (LiDAR was not avoiding lower obstacles so that needed to add ultrasonic for lower) -added nav2 algorithm for autonomous , planner, obstacles avoidance and so on.. -tested robot for obstacles avoidance

File: robot_ws/src/robot_description/urdf/robot.urdf.xacro (robot description, xacro)
@@ -31,11 +31,28 @@
   </link>
   <!-- ========================================================== -->
-  <!-- RPLIDAR A1                                                  -->
+  <!-- ULTRASONIC SENSOR                                          -->
+  <!-- ========================================================== -->
+  <link name="ultrasonic_link"/>
+  <joint name="ultrasonic_joint"
+         type="fixed">
+    <parent link="base_link"/>
+    <child link="ultrasonic_link"/>
+      <!-- Ultrasonic sensor position relative to base_link
+      X = 12.0 cm forward
+      Y = 6.0 cm left
+      Z = 8.6 cm above floor -->
+    <origin
+      xyz="0.120 0.060 0.086"
+      rpy="0 0 0"/>
+  </joint>
+  <!-- ========================================================== -->
+  <!-- RPLIDAR A1                                                 -->
   <!-- ========================================================== -->
   <link name="laser">
     <visual>
       <geometry>
-        <cylinder radius="0.035"
-                  length="0.04"/>
+        <cylinder
+          radius="0.035"
+          length="0.04"/>
       </geometry>
       <material name="black">
